File: electronics/led.brd (EAGLE design)
At the start: 8.9 x 5.1 mm, 4 parts

Commit message: RC0. Actual MOSTFET. Added sync pulse. Included LEDs
Other:
- outline, holes or cut-outs redrawn
Changed lines of the file:
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@@
 <layer number="44" name="Drills" color="7" fill="1" visible="no" active="yes"/>
 <layer number="45" name="Holes" color="7" fill="1" visible="no" active="yes"/>
-<layer number="46" name="Milling" color="3" fill="1" visible="no" active="yes"/>
+<layer number="46" name="Milling" color="3" fill="1" visible="yes" active="yes"/>
 <layer number="47" name="Measures" color="7" fill="1" visible="no" active="yes"/>
 <layer number="48" name="Document" color="7" fill="1" visible="yes" active="yes"/>
@@
 <wire x1="14.224" y1="1.27" x2="14.224" y2="6.35" width="0.4064" layer="20"/>
 <wire x1="14.224" y1="6.35" x2="5.334" y2="6.35" width="0.4064" layer="20"/>
+<wire x1="12.954" y1="3.81" x2="6.604" y2="3.81" width="0.4064" layer="46"/>
 </plain>
 <attributes>
