File: electronics/schematic.sch (EAGLE design)
At the start: 3 parts, among them Q1 MC-405

Commit message: Board getting close. Before switching Around
Parts:
- removed SV1: (no value), con-lstb:MA06-1
- added GND, GND2, LED+, LED-, RST, RXD, TEST, TXD, VCC, VCC2: TPTP15R, testpad:TPTP15R
- added Q3: SST201, transistor-fet:SST201
Connections:
- removed net VSS: SV1.2, U$1.4
- new net GND: GND.TP, Q3.S, U$1.4
- new net N$4: LED-.TP, Q3.D
- net LED: now also Q3.G
- net N$1: now also Q1.2; no longer Q1.1
- net N$2: now also Q1.1; no longer Q1.2
- net RST: now also RST.TP; no longer SV1.1
- net RXD: now also RXD.TP; no longer SV1.6
- net TEST: now also TEST.TP; no longer SV1.4
- net TXD: now also TXD.TP; no longer SV1.5
- net VCC: now also LED+.TP, VCC.TP; no longer SV1.3
Other:
- moved on the sheet: Q1

Commit message: Finished two layer design
Connections:
- net GND: now also GND2.TP
- net N$1: now also Q1.1; no longer Q1.2
- net N$2: now also Q1.2; no longer Q1.1
- net VCC: now also VCC2.TP
Other:
- moved on the sheet: GND2, VCC2
Changed lines of the file:
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@@
 <setting verticaltext="up"/>
 </settings>
-<grid distance="0.05" unitdist="inch" unit="inch" style="lines" multiple="1" display="no" altdistance="0.01" altunitdist="inch" altunit="inch"/>
+<grid distance="0.1" unitdist="inch" unit="inch" style="lines" multiple="1" display="yes" altdistance="0.01" altunitdist="inch" altunit="inch"/>
 <layers>
 <layer number="1" name="Top" color="4" fill="1" visible="no" active="no"/>
@@
 <instance part="LED+" gate="G$1" x="76.2" y="50.8" rot="R180"/>
 <instance part="LED-" gate="G$1" x="76.2" y="35.56"/>
-<instance part="VCC2" gate="G$1" x="-12.7" y="50.8" smashed="yes" rot="R90">
-<attribute name="NAME" x="-13.97" y="49.53" size="1.778" layer="95" rot="MR0"/>
-<attribute name="TP_SIGNAL_NAME" x="-11.43" y="52.07" size="1.778" layer="97" rot="R90"/>
-</instance>
-<instance part="GND2" gate="G$1" x="-12.7" y="46.99" smashed="yes" rot="R90">
-<attribute name="NAME" x="-13.97" y="45.72" size="1.778" layer="95" rot="MR0"/>
-<attribute name="TP_SIGNAL_NAME" x="-11.43" y="48.26" size="1.778" layer="97" rot="R90"/>
+<instance part="VCC2" gate="G$1" x="-12.7" y="33.02" smashed="yes" rot="R90">
+<attribute name="NAME" x="-13.97" y="31.75" size="1.778" layer="95" rot="MR0"/>
+<attribute name="TP_SIGNAL_NAME" x="-11.43" y="34.29" size="1.778" layer="97" rot="R90"/>
+</instance>
+<instance part="GND2" gate="G$1" x="-12.7" y="30.48" smashed="yes" rot="R90">
+<attribute name="NAME" x="-13.97" y="29.21" size="1.778" layer="95" rot="MR0"/>
+<attribute name="TP_SIGNAL_NAME" x="-11.43" y="31.75" size="1.778" layer="97" rot="R90"/>
 </instance>
 </instances>
@@
 <pinref part="U$1" gate="G$1" pin="5"/>
 <wire x1="-17.78" y1="71.12" x2="12.7" y2="71.12" width="0.1524" layer="91"/>
-<pinref part="Q1" gate="P" pin="2"/>
-<wire x1="-24.13" y1="72.39" x2="-17.78" y2="72.39" width="0.1524" layer="91"/>
+<pinref part="Q1" gate="P" pin="1"/>
+<wire x1="-24.13" y1="67.31" x2="-17.78" y2="72.39" width="0.1524" layer="91"/>
 </segment>
 </net>
@@
 <wire x1="12.7" y1="68.58" x2="-17.78" y2="68.58" width="0.1524" layer="91"/>
 <wire x1="-17.78" y1="68.58" x2="-17.78" y2="67.31" width="0.1524" layer="91"/>
-<pinref part="Q1" gate="P" pin="1"/>
-<wire x1="-24.13" y1="67.31" x2="-17.78" y2="67.31" width="0.1524" layer="91"/>
+<pinref part="Q1" gate="P" pin="2"/>
+<wire x1="-24.13" y1="72.39" x2="-17.78" y2="67.31" width="0.1524" layer="91"/>
 </segment>
 </net>
@@
 </segment>
 <segment>
-<wire x1="-10.16" y1="50.8" x2="10.16" y2="50.8" width="0.1524" layer="91"/>
-<label x="-7.62" y="50.8" size="1.778" layer="95"/>
+<pinref part="VCC2" gate="G$1" pin="TP"/>
+<wire x1="-10.16" y1="33.02" x2="2.54" y2="33.02" width="0.1524" layer="91"/>
+<label x="-7.62" y="33.02" size="1.778" layer="95"/>
 </segment>
 </net>
@@
 </segment>
 <segment>
-<wire x1="-10.16" y1="46.99" x2="10.16" y2="46.99" width="0.1524" layer="91"/>
-<label x="-7.62" y="46.99" size="1.778" layer="95"/>
-</segment>
-</net>
+<pinref part="GND2" gate="G$1" pin="TP"/>
+<wire x1="-10.16" y1="30.48" x2="2.54" y2="30.48" width="0.1524" layer="91"/>
+<label x="-7.62" y="30.48" size="1.778" layer="95"/>
+</segment>
+</net>

Commit message: Added bypass capacitor
Parts:
- added C1: (no value), resistor:C-EUC0805
Connections:
- net GND: now also C1.2
- net VCC: now also C1.1
Changed lines of the file:
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@@
 <part name="VCC2" library="testpad" deviceset="TP" device="TP15R" value="TPTP15R"/>
 <part name="GND2" library="testpad" deviceset="TP" device="TP15R" value="TPTP15R"/>
+<part name="C1" library="resistor" deviceset="C-EU" device="C0805"/>
 </parts>
 <sheets>
@@
 <attribute name="TP_SIGNAL_NAME" x="-11.43" y="31.75" size="1.778" layer="97" rot="R90"/>
 </instance>
+<instance part="C1" gate="G$1" x="-20.32" y="55.88"/>
 </instances>
 <busses>
@@
 <label x="-7.62" y="33.02" size="1.778" layer="95"/>
 </segment>
+<segment>
+<pinref part="C1" gate="G$1" pin="1"/>
+<wire x1="-20.32" y1="58.42" x2="-7.62" y2="58.42" width="0.1524" layer="91"/>
+<label x="-17.78" y="58.42" size="1.778" layer="95"/>
+</segment>
 </net>
 <net name="TXD" class="0">
@@
 <label x="-7.62" y="30.48" size="1.778" layer="95"/>
 </segment>
+<segment>
+<pinref part="C1" gate="G$1" pin="2"/>
+<wire x1="-20.32" y1="50.8" x2="-7.62" y2="50.8" width="0.1524" layer="91"/>
+<label x="-17.78" y="50.8" size="1.778" layer="95"/>
+</segment>
 </net>

Commit message: RC0. Actual MOSTFET. Added sync pulse. Included LEDs
Parts:
- removed GND2, LED+, LED-, VCC2: TPTP15R, testpad:TPTP15R
- removed Q1: MC-405, ROB:MC-405
- removed Q3: SST201, transistor-fet:SST201
- added LED1, LED2, LED3, LED4: (no value), led:LEDCHIP-LED0805
- added Q2: NX3008NBK, playafly:NX3008NBK
- added R1, R2, R3, R4: (no value), resistor:R-EU_M0805
- added SYNC0, SYNC1, VBAT+, VBAT-: TPTP15R, testpad:TPTP15R
- added U$2: AB26TRQ, playafly:AB26TRQ
Connections:
- removed net N$1: Q1.1, U$1.5
- removed net N$2: Q1.2, U$1.6
- new net N$5: LED2.C, R2.2
- new net N$6: LED3.C, R3.2
- new net N$7: LED4.C, R4.2
- new net N$8: Q2.D, R1.1, R2.1, R3.1, R4.1
- new net P2.0: SYNC0.TP, U$1.8
- new net XIN: U$1.6, U$2.1
- new net XOUT: U$1.5, U$2.2
- net GND: now also Q2.S, SYNC1.TP, U$2.3, VBAT-.TP; no longer GND2.TP, Q3.S
- net LED: now also Q2.G; no longer Q3.G
- net N$4: now also LED1.C, R1.2; no longer LED-.TP, Q3.D
- net RST: no longer U$1.7
- net VCC: now also LED1.A, LED2.A, LED3.A, LED4.A, U$1.7, VBAT+.TP; no longer LED+.TP, VCC2.TP
Other:
- note added: "Bypass Cap Electrolytic?"
- note added: "Launchpad ICSP Connection"
- note added: "Power connection 2 x CR2032 Parallel"
- moved on the sheet: C1, GND, RST, RXD, TEST, TXD, VCC

Commit message: new board design
Parts:
- added R5: (no value), resistor:R-EU_M0805
Connections:
- net LED: no longer U$1.13
- net RST: now also R5.1, U$1.7
- net VCC: now also R5.2; no longer U$1.7
- net XIN: now also U$2.2; no longer U$2.1
- net XOUT: now also U$2.1; no longer U$2.2
Changed lines of the file:
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@@
 <setting verticaltext="up"/>
 </settings>
-<grid distance="0.1" unitdist="inch" unit="inch" style="dots" multiple="1" display="yes" altdistance="0.05" altunitdist="inch" altunit="inch"/>
+<grid distance="0.1" unitdist="inch" unit="inch" style="lines" multiple="1" display="no" altdistance="0.01" altunitdist="inch" altunit="inch"/>
 <layers>
 <layer number="1" name="Top" color="4" fill="1" visible="no" active="no"/>
@@
 <part name="GND4" library="supply1" deviceset="GND" device=""/>
 <part name="P+3" library="supply1" deviceset="VCC" device=""/>
+<part name="R5" library="resistor" deviceset="R-EU_" device="M0805"/>
 </parts>
 <sheets>
@@
 </instance>
 <instance part="GND4" gate="1" x="99.06" y="10.16"/>
-<instance part="P+3" gate="VCC" x="50.8" y="68.58"/>
+<instance part="P+3" gate="VCC" x="43.18" y="68.58"/>
+<instance part="R5" gate="G$1" x="48.26" y="63.5" rot="R180"/>
 </instances>
 <busses>
@@
 </segment>
 <segment>
-<pinref part="U$2" gate="G$1" pin="2"/>
-<wire x1="66.04" y1="25.4" x2="72.898" y2="25.4" width="0.1524" layer="91"/>
+<pinref part="U$2" gate="G$1" pin="1"/>
+<wire x1="66.04" y1="10.16" x2="72.898" y2="25.4" width="0.1524" layer="91"/>
 <label x="66.04" y="25.4" size="1.778" layer="95"/>
 </segment>
@@
 </segment>
 <segment>
-<wire x1="66.04" y1="10.16" x2="73.406" y2="10.16" width="0.1524" layer="91"/>
-<pinref part="U$2" gate="G$1" pin="1"/>
+<wire x1="66.04" y1="25.4" x2="73.406" y2="10.16" width="0.1524" layer="91"/>
+<pinref part="U$2" gate="G$1" pin="2"/>
 <label x="66.04" y="10.16" size="1.778" layer="95"/>
 </segment>
@@
 <label x="19.05" y="8.89" size="1.778" layer="95"/>
 <pinref part="RST" gate="G$1" pin="TP"/>
+</segment>
+<segment>
+<pinref part="U$1" gate="G$1" pin="7"/>
+<wire x1="63.5" y1="63.5" x2="53.34" y2="63.5" width="0.1524" layer="91"/>
+<pinref part="R5" gate="G$1" pin="1"/>
+<label x="55.88" y="63.5" size="1.778" layer="95"/>
 </segment>
 </net>
@@
 </segment>
 <segment>
+<pinref part="R5" gate="G$1" pin="2"/>
 <pinref part="P+3" gate="VCC" pin="VCC"/>
-<wire x1="50.8" y1="66.04" x2="50.8" y2="63.5" width="0.1524" layer="91"/>
-<pinref part="U$1" gate="G$1" pin="7"/>
-<wire x1="63.5" y1="63.5" x2="50.8" y2="63.5" width="0.1524" layer="91"/>
+<wire x1="43.18" y1="63.5" x2="43.18" y2="66.04" width="0.1524" layer="91"/>
 </segment>
 </net>
@@
 <net name="LED" class="0">
 <segment>
-<pinref part="U$1" gate="G$1" pin="13"/>
-<wire x1="106.68" y1="60.96" x2="115.57" y2="60.96" width="0.1524" layer="91"/>
-<label x="109.22" y="60.96" size="1.778" layer="95"/>
-</segment>
-<segment>
 <wire x1="149.86" y1="27.94" x2="139.7" y2="27.94" width="0.1524" layer="91"/>
 <label x="142.24" y="27.94" size="1.778" layer="95"/>
 <pinref part="Q2" gate="A" pin="G"/>
 </segment>
-</net>
+<segment>
+<wire x1="106.68" y1="76.2" x2="115.57" y2="76.2" width="0.1524" layer="91"/>
+<label x="109.22" y="76.2" size="1.778" layer="95"/>
+</segment>
+</net>
